File: PCB/YonderDeep.brd (EAGLE design)
At the start: 67.3 x 58.1 mm, 10 parts

Commit message: AUV RaspberryPi PCB V2
Parts:
- moved U$1 0.63 mm to (59.7, 13.3)
Routing:
- net 3V3: track 164.8 -> 134.7 mm
- net SCL: track 113.5 -> 89.8 mm
- net GND: track 186.1 -> 171.9 mm
- net SDA: track 103.6 -> 96.3 mm
- net LM: track 62.9 -> 57.1 mm
- net BM: track 70.7 -> 66.9 mm
- net 5V: track 110.1 -> 106.3 mm
- net UART_TX: track 44.8 -> 43.8 mm
Other:
- board text added: "+"
- board text added: "-"
- board text added: "Yonder Deep V2 2/24/19"
- board text removed: "Yonder Deep V1 2/13/19"

Commit message: PCB V3
Parts:
- removed I2C_1: I2C_CONN, YonderDeep:1X04
- added CBST, C_IN2: 100 nF, Yonder_Deep_Library_Step_Down_Rasp:C0603K
- added COUT: 47 µF, Yonder_Deep_Library_Step_Down_Rasp:C1210K
- added C_IN: 22 µF, Yonder_Deep_Library_Step_Down_Rasp:C1206K
- added HYDRO: POWER_IN, YonderDeep:TERMINAL
- added IC1: MC78M09CDTRKG, SamacSys_Parts:TO229P991X238-4_3N
- added L1: XAL6030-332MEC, Yonder_Deep_Library_Step_Down_Rasp:XAL6030-122MEB
- added RFBT2: 10 kΩ, Yonder_Deep_Library_Step_Down_Rasp:RESC1005X40
- added RVBT: 56.2 kΩ, Yonder_Deep_Library_Step_Down_Rasp:R0402
- added U1: TPS565208DDCR, Yonder_Deep_Library_Step_Down_Rasp:SOT95P280X110-6N
- moved U$1 31.0 mm to (59.7, 44.3), turned to 270 degrees
- moved IMU 9.04 mm to (26.2, 23.4)
- renumbered 5V_IN to BATTERY, I2C_2 to I2C
Connections:
- new net N$1: CBST.2, U1.6
- new net N$2: CBST.1, L1.1, U1.2
- new net N$3: RFBT2.1, RVBT.1, U1.4
- new net VIN: BATTERY.+, C_IN.1, C_IN2.1, IC1.1, U1.3, U1.5
- new net VOUT_HYDRO: HYDRO.+, IC1.3
- net 3V3: no longer I2C_1.VCC
- net 5V: now also COUT.1, L1.2, RVBT.2; no longer BATTERY.+
- net GND: now also COUT.2, C_IN.2, C_IN2.2, HYDRO.-, IC1.4, RFBT2.2, U1.1; no longer I2C_1.GND
- net SCL: no longer I2C_1.SCL
- net SDA: no longer I2C_1.SDA
Routing:
- net GND: track 171.9 -> 229.7 mm, vias 0 -> 1
- net VIN: track 0.00 -> 53.9 mm
- net N$2: track 0.00 -> 26.6 mm
- net FM: track 56.0 -> 77.9 mm
- net 5V: track 106.3 -> 124.3 mm, vias 0 -> 3
- net VOUT_HYDRO: track 0.00 -> 16.9 mm
- net 3V3: track 134.7 -> 146.1 mm
- net N$1: track 0.00 -> 8.73 mm
- net N$3: track 0.00 -> 8.61 mm
- net BM: track 66.9 -> 60.7 mm
- net LM: track 57.1 -> 60.9 mm
- net UART_RX: track 41.8 -> 39.1 mm
- net SDA: track 96.3 -> 98.2 mm
- net UART_TX: track 43.8 -> 42.6 mm
- net SCL: track 89.8 -> 90.4 mm
- removed copper zone on layer 1, net GND
- removed copper zone on layer 16, net GND
Other:
- board text added: "Yonder Deep V3 4/17/19"
- board text removed: "Yonder Deep V2 2/24/19"
