File: PCB/YonderDeep.sch (EAGLE design)
At the start: 10 parts

Commit message: PCB V3
Parts:
- removed I2C_1: I2C_CONN, YonderDeep:I2C_CONN
- added CBST, C_IN2: 100 nF, Yonder_Deep_Library_Step_Down_Rasp:C0603C104Z3VACTU
- added COUT: 47 µF, Yonder_Deep_Library_Step_Down_Rasp:TMK325ABJ476MM-P
- added C_IN: 22 µF, Yonder_Deep_Library_Step_Down_Rasp:C3216JB1V226M160AC
- added HYDRO: POWER_IN, YonderDeep:POWER_IN
- added IC1: MC78M09CDTRKG, SamacSys_Parts:MC78M09CDTRKG
- added L1: XAL6030-332MEC, Yonder_Deep_Library_Step_Down_Rasp:XAL6030-332MEC
- added RFBT2: 10 kΩ, Yonder_Deep_Library_Step_Down_Rasp:RMCF0402FT10K0
- added RVBT: 56.2 kΩ, Yonder_Deep_Library_Step_Down_Rasp:AC0402FR-0756K2L
- added U1: TPS565208DDCR, Yonder_Deep_Library_Step_Down_Rasp:TPS565208DDCR
- renumbered 5V_IN to BATTERY, I2C_2 to I2C
Connections:
- new net N$1: CBST.2, U1.VBST
- new net N$2: CBST.1, L1.1, U1.SW
- new net N$3: RFBT2.1, RVBT.1, U1.VFB
- new net VIN: BATTERY.+, C_IN.1, C_IN2.1, IC1.INPUT, U1.EN, U1.VIN
- new net VOUT_HYDRO: HYDRO.+, IC1.OUTPUT
- net 3V3: no longer I2C_1.VCC
- net 5V: now also COUT.1, L1.2, RVBT.2; no longer BATTERY.+
- net GND: now also COUT.2, C_IN.2, C_IN2.2, HYDRO.-, IC1.GROUND, RFBT2.2, U1.GND; no longer I2C_1.GND
- net SCL: no longer I2C_1.SCL
- net SDA: no longer I2C_1.SDA
